Commit message: Try various cases for gazebo

File: bogie_mobile_robot_description/urdf/gazebo.urdf.xacro (robot description, xacro)
@@ -2,44 +2,44 @@
 <robot xmlns:xacro="http://wiki.ros.org/xacro">
     <gazebo reference="l_wheel">
-        <mu value="200.0"/>
+        <mu1 value="200.0"/>
         <mu2 value="200.0"/>
         <kp value="10000000.0" />
         <kd value="1.0" />
-        <minDepth>0.01</minDepth>
+        <minDepth>0.0</minDepth>
     </gazebo>
     <gazebo reference="r_wheel">
-        <mu value="200.0"/>
+        <mu1 value="200.0"/>
         <mu2 value="200.0"/>
         <kp value="10000000.0" />
         <kd value="1.0" />
-        <minDepth>0.01</minDepth>
+        <minDepth>0.0</minDepth>
     </gazebo>
     <gazebo reference="l_rear_caster_wheel">
-        <mu value="1"/>
+        <mu1 value="1"/>
         <mu2 value="1"/>
         <kp value="10000000.0"/>
         <kd value="1.0"/>
-        <minDepth>0.01</minDepth>
+        <minDepth>0.0</minDepth>
     </gazebo>
     <gazebo reference="r_rear_caster_wheel">
-        <mu value="1"/>
+        <mu1 value="1"/>
         <mu2 value="1"/>
         <kp value="10000000.0"/>
         <kd value="1.0"/>
-        <minDepth>0.01</minDepth>
+        <minDepth>0.0</minDepth>
     </gazebo>
     <gazebo reference="l_front_caster_wheel">
-        <mu value="1"/>
+        <mu1 value="1"/>
         <mu2 value="1"/>
         <kp value="10000000.0"/>
         <kd value="1.0"/>
-        <minDepth>0.01</minDepth>
+        <minDepth>0.0</minDepth>
     </gazebo>
     <gazebo reference="r_front_caster_wheel">
-        <mu value="1"/>
+        <mu1 value="1"/>
         <mu2 value="1"/>
         <kp value="10000000.0"/>
         <kd value="1.0"/>
-        <minDepth>0.01</minDepth>
+        <minDepth>0.0</minDepth>
     </gazebo>
     <gazebo>
@@ -51,3 +51,11 @@
         </plugin>
     </gazebo>
+    <!-- <gazebo>
+        <plugin name="differential_drive_controller" filename="libgazebo_ros_diff_drive.so">
+            <leftJoint>l_wheel_joint</leftJoint>
+            <rightJoint>r_wheel_joint</rightJoint>
+            <wheelSeparation>0.8</wheelSeparation>
+            <wheelDiameter>0.2</wheelDiameter>
+        </plugin>
+    </gazebo> -->
 </robot>

File: bogie_mobile_robot_description/urdf/robot.urdf.xacro (robot description, xacro)
@@ -75,6 +75,6 @@
                 <mass value="2.0"/>
                 <origin xyz="0 0 0" rpy="${pi/2} 0 0"/>
-                <!-- <xacro:cylinder_inertia m="2.0" r="0.1" h="0.06"/> -->
-                <inertia ixx="0.2" ixy="0.0" ixz="0.0" iyy="0.2" iyz="0.0" izz="0.2"/>
+                <xacro:cylinder_inertia m="2.0" r="0.1" h="0.06"/>
+                <!-- <inertia ixx="0.2" ixy="0.0" ixz="0.0" iyy="0.2" iyz="0.0" izz="0.2"/> -->
             </inertial>
         </link>
@@ -133,5 +133,5 @@
             <parent link="${prefix}_rear_caster_rotate"/>
             <child link="${prefix}_rear_caster_wheel"/>
-            <origin xyz="-0.015 0 -0.09" rpy="0 0 0"/>
+            <origin xyz="-0.02 0 -0.09" rpy="0 0 0"/>
             <axis xyz="0 1 0"/>
         </joint>
@@ -187,5 +187,5 @@
             <parent link="${prefix}_front_caster_rotate"/>
             <child link="${prefix}_front_caster_wheel"/>
-            <origin xyz="-0.015 0 -0.09" rpy="0 0 0"/>
+            <origin xyz="-0.02 0 -0.09" rpy="0 0 0"/>
             <axis xyz="0 1 0"/>
         </joint>

Commit message: Bug fixed

File: bogie_mobile_robot_description/urdf/gazebo.urdf.xacro (robot description, xacro)
@@ -49,4 +49,5 @@
             <controlPeriod>0.001</controlPeriod>
             <legacyModeNS>false</legacyModeNS>
+            <eStopTopic>emergency_stop</eStopTopic>
         </plugin>
     </gazebo>

File: bogie_mobile_robot_description/urdf/robot.urdf.xacro (robot description, xacro)
@@ -22,7 +22,7 @@
         </collision>
         <inertial>
-            <mass value="100.0"/>
+            <mass value="60.0"/>
             <origin xyz="0 0 0" rpy="0 0 0"/>
-            <xacro:box_inertia m="100.0" x="1.0" y="0.55" z="0.20"/>
+            <xacro:box_inertia m="60.0" x="1.0" y="0.55" z="0.20"/>
         </inertial>
     </link>
@@ -47,15 +47,16 @@
             </collision>
             <inertial>
-                <mass value="2.0"/>
+                <mass value="1.0"/>
                 <origin xyz="0 ${-dir*0.01} 0" rpy="${pi/2} 0 0"/>
-                <xacro:cylinder_inertia m="2.0" r="0.03" h="0.08"/>
+                <!-- <xacro:cylinder_inertia m="1.0" r="0.03" h="0.08"/> -->
+                <inertia ixx="1.0" ixy="0.0" ixz="0.0" iyy="1.0" iyz="0.0" izz="1.0"/>
             </inertial>
         </link>
-        <joint name="${prefix}_bogie_suspension_joint" type="revolute">
+        <joint name="${prefix}_bogie_suspension_joint" type="continuous">
             <parent link="base_link"/>
             <child link="${prefix}_bogie_suspension"/>
             <origin xyz="-0.25 ${dir*0.36} 0" rpy="0 0 0"/>
             <axis xyz="0 1 0"/>
-            <limit effort="1000" velocity="0.1" lower="${-pi}" upper="${pi}"/>
+            <!-- <limit effort="10" velocity="3.0" lower="${-pi}" upper="${pi}"/> -->
         </joint>
         <link name="${prefix}_wheel">
@@ -84,4 +85,5 @@
             <origin xyz="0.25 ${dir*0.01} -0.05" rpy="0 0 0"/>
             <axis xyz="0 1 0"/>
+            <limit effort="1000000" velocity="20.0"/>
         </joint>
         <xacro:insert_velocity_transmission name="${prefix}_wheel_joint"/>
@@ -100,7 +102,7 @@
             </collision>
             <inertial>
-                <mass value="2.0"/>
+                <mass value="0.1"/>
                 <origin xyz="0 0 0" rpy="0 0 0"/>
-                <xacro:cylinder_inertia m="2.0" r="0.03" h="0.03"/>
+                <xacro:cylinder_inertia m="0.1" r="0.03" h="0.03"/>
             </inertial>
         </link>
@@ -125,7 +127,7 @@
             </collision>
             <inertial>
-                <mass value="2.0"/>
+                <mass value="0.1"/>
                 <origin xyz="0 0 0" rpy="${pi/2} 0 0"/>
-                <xacro:cylinder_inertia m="2.0" r="0.06" h="0.04"/>
+                <xacro:cylinder_inertia m="0.1" r="0.06" h="0.04"/>
             </inertial>
         </link>
@@ -135,4 +137,5 @@
             <origin xyz="-0.02 0 -0.09" rpy="0 0 0"/>
             <axis xyz="0 1 0"/>
+            <limit effort="1000000" velocity="20.0"/>
         </joint>
     </xacro:macro>
@@ -154,7 +157,7 @@
             </collision>
             <inertial>
-                <mass value="2.0"/>
+                <mass value="0.1"/>
                 <origin xyz="0 0 0" rpy="0 0 0"/>
-                <xacro:cylinder_inertia m="2.0" r="0.03" h="0.03"/>
+                <xacro:cylinder_inertia m="0.1" r="0.03" h="0.03"/>
             </inertial>
         </link>
@@ -179,7 +182,7 @@
             </collision>
             <inertial>
-                <mass value="2.0"/>
+                <mass value="0.1"/>
                 <origin xyz="0 0 0" rpy="${pi/2} 0 0"/>
-                <xacro:cylinder_inertia m="2.0" r="0.06" h="0.04"/>
+                <xacro:cylinder_inertia m="0.1" r="0.06" h="0.04"/>
             </inertial>
         </link>
